File: Hardware/LilyPixel.brd (EAGLE design)
At the start: 20 x 20 mm, 15 parts

Commit message: added regular fiducials
Parts:
- FID1, FID2: value FIDUCIALUFIDUCIAL -> FIDUCIAL1X2; device SparkFun-Aesthetics:MICRO-FIDUCIAL -> SparkFun-Aesthetics:FIDUCIAL-1X2
- moved FID1 13.3 mm to (-3.81, 6.86)
- moved FID2 12.8 mm to (3.81, -6.86)
