File: Production Files/LilyPixel-Panel-v11.brd (EAGLE design)
At the start: 129.5 x 129.5 mm, 253 parts, among them U1 WS2811, U10 WS2811, U11 WS2811, U12 WS2811, U13 WS2811, U14 WS2811, U15 WS2811, U16 WS2811, U17 WS2811, U18 WS2811, U19 WS2811, U2 WS2811, U20 WS2811, U21 WS2811, U22 WS2811, U23 WS2811, U24 WS2811, U25 WS2811, U3 WS2811, U4 WS2811, U5 WS2811, U6 WS2811, U7 WS2811, U8 WS2811, U9 WS2811

Commit message: created panel v11
Parts:
- removed E$3, E$6: (no value), SparkFun-Aesthetics:FIDUCIAL-1X2
- removed U$100, U$101, U$102, U$105, U$106, U$107, U$108, U$109, U$110, U$113, U$114, U$115, U$116, U$117, U$118, U$121, U$122, U$123, U$124, U$125, U$126, U$129, U$130, U$131, U$132, U$133, U$134, U$137, U$138, U$139, U$140, U$141, U$142, U$145, U$146, U$147, U$148, U$149, U$150, U$153, U$154, U$155, U$156, U$157, U$158, U$161, U$162, U$163, U$164, U$165, U$166, U$169, U$170, U$171, U$172, U$173, U$174, U$177, U$178, U$179, U$180, U$181, U$182, U$185, U$186, U$187, U$188, U$189, U$190, U$193, U$194, U$195, U$196, U$197, U$198, U$51, U$52, U$53, U$54, U$57, U$58, U$59, U$60, U$61, U$62, U$65, U$66, U$67, U$68, U$69, U$70, U$73, U$74, U$75, U$76, U$77, U$78, U$81, U$82, U$83, U$84, U$85, U$86, U$89, U$90, U$91, U$92, U$93, U$94, U$97, U$98, U$99: SEWTAP6, LilyPad-Wearables:PETAL-SMALL-2SIDE
- removed U$103, U$111, U$119, U$127, U$135, U$143, U$151, U$159, U$167, U$175, U$183, U$191, U$199, U$55, U$63, U$71, U$79, U$87, U$95: LOGO-LPL, LilyPad-Wearables:LOGO-L
- removed U$104, U$112, U$120, U$128, U$136, U$144, U$152, U$160, U$168, U$176, U$184, U$192, U$200, U$56, U$64, U$72, U$80, U$88, U$96: LOGO-LPLP, LilyPad-Wearables:LOGO-LILYPAD
- removed U1, U10, U11, U12, U13, U14, U15, U16, U17, U18, U19, U2, U20, U21, U22, U23, U24, U25, U3, U4, U5, U6, U7, U8, U9: WS2811, SparkFun-LED:LED-TRICOLOR-5050-IC
- added D1, D10, D11, D12, D13, D14, D15, D16, D17, D18, D19, D2, D20, D21, D22, D23, D24, D25, D3, D4, D5, D6, D7, D8, D9: WS2812B, SparkFun-LED:WS2812B
- added E$4, E$5: (no value), SparkFun-Aesthetics:FIDUCIAL-1X2
- added FID1, FID10, FID11, FID12, FID13, FID14, FID15, FID16, FID17, FID18, FID19, FID2, FID20, FID21, FID22, FID23, FID24, FID25, FID26, FID27, FID28, FID29, FID3, FID30, FID31, FID32, FID33, FID34, FID35, FID36, FID37, FID38, FID39, FID4, FID40, FID41, FID42, FID43, FID44, FID45, FID46, FID47, FID48, FID49, FID5, FID50, FID6, FID7, FID8, FID9: FIDUCIAL1X2, SparkFun-Aesthetics:FIDUCIAL-1X2
- added JP1, JP10, JP100, JP101, JP102, JP103, JP104, JP105, JP106, JP107, JP108, JP109, JP11, JP110, JP111, JP112, JP113, JP114, JP115, JP116, JP117, JP118, JP119, JP12, JP120, JP121, JP122, JP123, JP124, JP125, JP126, JP127, JP128, JP129, JP13, JP130, JP131, JP132, JP133, JP134, JP135, JP136, JP137, JP138, JP139, JP14, JP140, JP141, JP142, JP143, JP144, JP145, JP146, JP147, JP148, JP149, JP15, JP150, JP16, JP17, JP18, JP19, JP2, JP20, JP21, JP22, JP23, JP24, JP25, JP26, JP27, JP28, JP29, JP3, JP30, JP31, JP32, JP33, JP34, JP35, JP36, JP37, JP38, JP39, JP4, JP40, JP41, JP42, JP43, JP44, JP45, JP46, JP47, JP48, JP49, JP5, JP50, JP51, JP52, JP53, JP54, JP55, JP56, JP57, JP58, JP59, JP6, JP60, JP61, JP62, JP63, JP64, JP65, JP66, JP67, JP68, JP69, JP7, JP70, JP71, JP72, JP73, JP74, JP75, JP76, JP77, JP78, JP79, JP8, JP80, JP81, JP82, JP83, JP84, JP85, JP86, JP87, JP88, JP89, JP9, JP90, JP91, JP92, JP93, JP94, JP95, JP96, JP97, JP98, JP99: SEWTAP6, LilyPad-Wearables:PETAL-SMALL-2SIDE
- added LOGO1, LOGO11, LOGO13, LOGO15, LOGO17, LOGO19, LOGO21, LOGO23, LOGO25, LOGO27, LOGO29, LOGO3, LOGO31, LOGO33, LOGO35, LOGO37, LOGO39, LOGO41, LOGO43, LOGO45, LOGO47, LOGO49, LOGO5, LOGO7, LOGO9: OSHW-LOGOS, SparkFun-Aesthetics:OSHW-LOGO-S
- added LOGO10, LOGO12, LOGO14, LOGO16, LOGO18, LOGO2, LOGO20, LOGO22, LOGO24, LOGO26, LOGO28, LOGO30, LOGO32, LOGO34, LOGO36, LOGO38, LOGO4, LOGO40, LOGO42, LOGO44, LOGO46, LOGO48, LOGO50, LOGO6, LOGO8: SFE_LOGO_FLAME.1_INCH, SparkFun-Aesthetics:SFE_LOGO_FLAME_.1
- E$1: device SparkFun-Aesthetics:FIDUCIAL-1.5X3 -> SparkFun-Retired:FIDUCIAL-1.5X3
- U$10, U$12, U$14, U$18, U$20, U$22, U$26, U$28, U$3, U$30, U$34, U$36, U$38, U$42, U$44, U$46, U$5, U$50, U$7: value SEWTAP6 -> LOGO-LPLP; device LilyPad-Wearables:PETAL-SMALL-2SIDE -> LilyPad-Wearables:LOGO-LILYPAD
- U$11, U$13, U$17, U$19, U$2, U$21, U$25, U$27, U$29, U$33, U$35, U$37, U$4, U$41, U$43, U$45, U$49, U$6, U$9: value SEWTAP6 -> LOGO-LPL; device LilyPad-Wearables:PETAL-SMALL-2SIDE -> LilyPad-Wearables:LOGO-L
- moved U$34 104.2 mm to (41.9, 87.6), flipped to the bottom, turned to 0 degrees
- moved U$49 101.3 mm to (110.5, 106.2), turned to 0 degrees
- moved U$32 97.0 mm to (19.1, 87.6)
- moved U$48 97.0 mm to (87.6, 110.5)
- moved U$31 96.8 mm to (19.1, 83.3)
- moved U$47 96.8 mm to (87.6, 106.2)
- moved U$50 95.3 mm to (110.5, 110.5), flipped to the bottom, turned to 0 degrees
- moved U$33 92.1 mm to (41.9, 83.3), turned to 0 degrees
- moved U$46 88.8 mm to (64.8, 110.5), flipped to the bottom
- moved U$35 79.9 mm to (64.8, 83.3), turned to 0 degrees
- moved U$38 79.4 mm to (87.6, 87.6), flipped to the bottom
- moved U$36 75.8 mm to (64.8, 87.6), flipped to the bottom, turned to 0 degrees
- moved U$9 75.1 mm to (110.5, 14.7), turned to 0 degrees
- moved U$45 72.9 mm to (64.8, 106.2), turned to 0 degrees
- moved U$42 72.6 mm to (19.1, 110.5), flipped to the bottom, turned to 0 degrees
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Connections:
- removed net DI: U$2.1, U$4.1, U1.2
- removed net DO: U$3.1, U$5.1, U1.1
- new net DI25: D25.4, JP146.1, JP150.1
- new net DO25: D25.2, JP148.1, JP149.1
- net DI1: now also D1.4, JP5.1, JP6.1; no longer U$11.1, U$9.1, U2.2
- net DI10: now also D10.4, JP56.1, JP60.1; no longer U$81.1, U$83.1, U11.2
- net DI11: now also D11.4, JP62.1, JP66.1; no longer U$89.1, U$91.1, U12.2
- net DI12: now also D12.4, JP68.1, JP72.1; no longer U$97.1, U$99.1, U13.2
- net DI13: now also D13.4, JP74.1, JP78.1; no longer U$105.1, U$107.1, U14.2
- net DI14: now also D14.4, JP80.1, JP84.1; no longer U$113.1, U$115.1, U15.2
- net DI15: now also D15.4, JP86.1, JP90.1; no longer U$121.1, U$123.1, U16.2
- net DI16: now also D16.4, JP92.1, JP96.1; no longer U$129.1, U$131.1, U17.2
- net DI17: now also D17.4, JP102.1, JP98.1; no longer U$137.1, U$139.1, U18.2
- net DI18: now also D18.4, JP104.1, JP108.1; no longer U$145.1, U$147.1, U19.2
- net DI19: now also D19.4, JP110.1, JP114.1; no longer U$153.1, U$155.1, U20.2
- net DI2: now also D2.4, JP12.1, JP8.1; no longer U$17.1, U$19.1, U3.2
- net DI20: now also D20.4, JP116.1, JP120.1; no longer U$161.1, U$163.1, U21.2
- net DI21: now also D21.4, JP122.1, JP126.1; no longer U$169.1, U$171.1, U22.2
- net DI22: now also D22.4, JP128.1, JP132.1; no longer U$177.1, U$179.1, U23.2
- net DI23: now also D23.4, JP134.1, JP138.1; no longer U$185.1, U$187.1, U24.2
- net DI24: now also D24.4, JP140.1, JP144.1; no longer U$193.1, U$195.1, U25.2
- net DI3: now also D3.4, JP14.1, JP18.1; no longer U$25.1, U$27.1, U4.2
- net DI4: now also D4.4, JP20.1, JP24.1; no longer U$33.1, U$35.1, U5.2
- net DI5: now also D5.4, JP26.1, JP30.1; no longer U$41.1, U$43.1, U6.2
- net DI6: now also D6.4, JP32.1, JP36.1; no longer U$49.1, U$51.1, U7.2
- net DI7: now also D7.4, JP38.1, JP42.1; no longer U$57.1, U$59.1, U8.2
- net DI8: now also D8.4, JP44.1, JP48.1; no longer U$65.1, U$67.1, U9.2
- net DI9: now also D9.4, JP50.1, JP54.1; no longer U$73.1, U$75.1, U10.2
- net DO1: now also D1.2, JP1.1, JP2.1; no longer U$10.1, U$12.1, U2.1
- net DO10: now also D10.2, JP58.1, JP59.1; no longer U$82.1, U$84.1, U11.1
- net DO11: now also D11.2, JP64.1, JP65.1; no longer U$90.1, U$92.1, U12.1
- net DO12: now also D12.2, JP70.1, JP71.1; no longer U$100.1, U$98.1, U13.1
- net DO13: now also D13.2, JP76.1, JP77.1; no longer U$106.1, U$108.1, U14.1
- net DO14: now also D14.2, JP82.1, JP83.1; no longer U$114.1, U$116.1, U15.1
- net DO15: now also D15.2, JP88.1, JP89.1; no longer U$122.1, U$124.1, U16.1
- net DO16: now also D16.2, JP94.1, JP95.1; no longer U$130.1, U$132.1, U17.1
- net DO17: now also D17.2, JP100.1, JP101.1; no longer U$138.1, U$140.1, U18.1
- net DO18: now also D18.2, JP106.1, JP107.1; no longer U$146.1, U$148.1, U19.1
- net DO19: now also D19.2, JP112.1, JP113.1; no longer U$154.1, U$156.1, U20.1
- net DO2: now also D2.2, JP10.1, JP11.1; no longer U$18.1, U$20.1, U3.1
- net DO20: now also D20.2, JP118.1, JP119.1; no longer U$162.1, U$164.1, U21.1
- net DO21: now also D21.2, JP124.1, JP125.1; no longer U$170.1, U$172.1, U22.1
- net DO22: now also D22.2, JP130.1, JP131.1; no longer U$178.1, U$180.1, U23.1
- net DO23: now also D23.2, JP136.1, JP137.1; no longer U$186.1, U$188.1, U24.1
- net DO24: now also D24.2, JP142.1, JP143.1; no longer U$194.1, U$196.1, U25.1
- net DO3: now also D3.2, JP16.1, JP17.1; no longer U$26.1, U$28.1, U4.1
- net DO4: now also D4.2, JP22.1, JP23.1; no longer U$34.1, U$36.1, U5.1
- net DO5: now also D5.2, JP28.1, JP29.1; no longer U$42.1, U$44.1, U6.1
- net DO6: now also D6.2, JP34.1, JP35.1; no longer U$50.1, U$52.1, U7.1
- net DO7: now also D7.2, JP40.1, JP41.1; no longer U$58.1, U$60.1, U8.1
- net DO8: now also D8.2, JP46.1, JP47.1; no longer U$66.1, U$68.1, U9.1
- net DO9: now also D9.2, JP52.1, JP53.1; no longer U$74.1, U$76.1, U10.1
- net GND: now also C2.2, D1.3, JP3.1; no longer C1.2, U$7.1, U1.6
- net GND1: now also C1.2, D2.3, JP9.1; no longer C2.2, U$14.1, U2.6
- net GND10: now also D11.3, JP63.1; no longer U$86.1, U11.6
- net GND11: now also D12.3, JP69.1; no longer U$94.1, U12.6
- net GND12: now also D13.3, JP75.1; no longer U$102.1, U13.6
- net GND13: now also D14.3, JP81.1; no longer U$110.1, U14.6
- net GND14: now also D15.3, JP87.1; no longer U$118.1, U15.6
- net GND15: now also D16.3, JP93.1; no longer U$126.1, U16.6
- net GND16: now also D17.3, JP99.1; no longer U$134.1, U17.6
- net GND17: now also D18.3, JP105.1; no longer U$142.1, U18.6
- net GND18: now also D19.3, JP111.1; no longer U$150.1, U19.6
- net GND19: now also D20.3, JP117.1; no longer U$158.1, U20.6
- net GND2: now also D3.3, JP15.1; no longer U$22.1, U3.6
- net GND20: now also D21.3, JP123.1; no longer U$166.1, U21.6
- net GND21: now also D22.3, JP129.1; no longer U$174.1, U22.6
- net GND22: now also D23.3, JP135.1; no longer U$182.1, U23.6
- net GND23: now also D24.3, JP141.1; no longer U$190.1, U24.6
- net GND24: now also D25.3, JP147.1; no longer U$198.1, U25.6
- net GND3: now also D4.3, JP21.1; no longer U$30.1, U4.6
- net GND4: now also D5.3, JP27.1; no longer U$38.1, U5.6
- net GND5: now also D6.3, JP33.1; no longer U$46.1, U6.6
- net GND6: now also D7.3, JP39.1; no longer U$54.1, U7.6
- net GND7: now also D8.3, JP45.1; no longer U$62.1, U8.6
- net GND8: now also D9.3, JP51.1; no longer U$70.1, U9.6
- net GND9: now also D10.3, JP57.1; no longer U$78.1, U10.6
- net VCC: now also C2.1, D1.1, JP4.1; no longer C1.1, U$6.1, U1.3, U1.5
- net VCC1: now also C1.1, D2.1, JP7.1; no longer C2.1, U$13.1, U2.3, U2.5
- net VCC10: now also D11.1, JP61.1; no longer U$85.1, U11.3, U11.5
- net VCC11: now also D12.1, JP67.1; no longer U$93.1, U12.3, U12.5
- net VCC12: now also D13.1, JP73.1; no longer U$101.1, U13.3, U13.5
- net VCC13: now also D14.1, JP79.1; no longer U$109.1, U14.3, U14.5
- net VCC14: now also D15.1, JP85.1; no longer U$117.1, U15.3, U15.5
- net VCC15: now also D16.1, JP91.1; no longer U$125.1, U16.3, U16.5
- net VCC16: now also D17.1, JP97.1; no longer U$133.1, U17.3, U17.5
- net VCC17: now also D18.1, JP103.1; no longer U$141.1, U18.3, U18.5
- net VCC18: now also D19.1, JP109.1; no longer U$149.1, U19.3, U19.5
- net VCC19: now also D20.1, JP115.1; no longer U$157.1, U20.3, U20.5
- net VCC2: now also D3.1, JP13.1; no longer U$21.1, U3.3, U3.5
- net VCC20: now also D21.1, JP121.1; no longer U$165.1, U21.3, U21.5
- net VCC21: now also D22.1, JP127.1; no longer U$173.1, U22.3, U22.5
- net VCC22: now also D23.1, JP133.1; no longer U$181.1, U23.3, U23.5
- net VCC23: now also D24.1, JP139.1; no longer U$189.1, U24.3, U24.5
- net VCC24: now also D25.1, JP145.1; no longer U$197.1, U25.3, U25.5
- net VCC3: now also D4.1, JP19.1; no longer U$29.1, U4.3, U4.5
- net VCC4: now also D5.1, JP25.1; no longer U$37.1, U5.3, U5.5
- net VCC5: now also D6.1, JP31.1; no longer U$45.1, U6.3, U6.5
- net VCC6: now also D7.1, JP37.1; no longer U$53.1, U7.3, U7.5
- net VCC7: now also D8.1, JP43.1; no longer U$61.1, U8.3, U8.5
- net VCC8: now also D9.1, JP49.1; no longer U$69.1, U9.3, U9.5
- net VCC9: now also D10.1, JP55.1; no longer U$77.1, U10.3, U10.5
Routing:
- net DI: track 23.8 -> 0.00 mm
- net DO: track 21.7 -> 0.00 mm, vias 2 -> 0
- net DO25: track 0.00 -> 17.7 mm
- net DI25: track 0.00 -> 15.9 mm, vias 0 -> 1
- net DI16: track 23.8 -> 15.9 mm, vias 0 -> 1
- net DI17: track 23.8 -> 15.9 mm, vias 0 -> 1
- net DI15: track 23.8 -> 15.9 mm, vias 0 -> 1
- net DI12: track 23.8 -> 15.9 mm, vias 0 -> 1
- net DI11: track 23.8 -> 15.9 mm, vias 0 -> 1
- net DI21: track 23.8 -> 15.9 mm, vias 0 -> 1
- net DI19: track 23.8 -> 15.9 mm, vias 0 -> 1
- net DI18: track 23.8 -> 15.9 mm, vias 0 -> 1
- net DI6: track 23.8 -> 15.9 mm, vias 0 -> 1
- net DI13: track 23.8 -> 15.9 mm, vias 0 -> 1
- net DI22: track 23.8 -> 15.9 mm, vias 0 -> 1
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Other:
- board text added: "v11"
- board text removed: "v10"

Commit message: made it a giant
Parts:
- added C26, C27, C28, C29, C30, C31, C32, C33, C34, C35, C36, C37, C38, C39, C40, C41, C42, C43, C44, C45, C46, C47, C48, C49, C50: 0.1uF, SparkFun-Capacitors:0603-CAP
- added D26, D27, D28, D29, D30, D31, D32, D33, D34, D35, D36, D37, D38, D39, D40, D41, D42, D43, D44, D45, D46, D47, D48, D49, D50: WS2812B, SparkFun-LED:WS2812B
- added E$2, E$3: (no value), SparkFun-Aesthetics:FIDUCIAL-1X2
- added E$6: (no value), SparkFun-Retired:FIDUCIAL-1.5X3
- added FID100, FID51, FID52, FID53, FID54, FID55, FID56, FID57, FID58, FID59, FID60, FID61, FID62, FID63, FID64, FID65, FID66, FID67, FID68, FID69, FID70, FID71, FID72, FID73, FID74, FID75, FID76, FID77, FID78, FID79, FID80, FID81, FID82, FID83, FID84, FID85, FID86, FID87, FID88, FID89, FID90, FID91, FID92, FID93, FID94, FID95, FID96, FID97, FID98, FID99: FIDUCIAL1X2, SparkFun-Aesthetics:FIDUCIAL-1X2
- added JP151, JP152, JP153, JP154, JP155, JP156, JP157, JP158, JP159, JP160, JP161, JP162, JP163, JP164, JP165, JP166, JP167, JP168, JP169, JP170, JP171, JP172, JP173, JP174, JP175, JP176, JP177, JP178, JP179, JP180, JP181, JP182, JP183, JP184, JP185, JP186, JP187, JP188, JP189, JP190, JP191, JP192, JP193, JP194, JP195, JP196, JP197, JP198, JP199, JP200, JP201, JP202, JP203, JP204, JP205, JP206, JP207, JP208, JP209, JP210, JP211, JP212, JP213, JP214, JP215, JP216, JP217, JP218, JP219, JP220, JP221, JP222, JP223, JP224, JP225, JP226, JP227, JP228, JP229, JP230, JP231, JP232, JP233, JP234, JP235, JP236, JP237, JP238, JP239, JP240, JP241, JP242, JP243, JP244, JP245, JP246, JP247, JP248, JP249, JP250, JP251, JP252, JP253, JP254, JP255, JP256, JP257, JP258, JP259, JP260, JP261, JP262, JP263, JP264, JP265, JP266, JP267, JP268, JP269, JP270, JP271, JP272, JP273, JP274, JP275, JP276, JP277, JP278, JP279, JP280, JP281, JP282, JP283, JP284, JP285, JP286, JP287, JP288, JP289, JP290, JP291, JP292, JP293, JP294, JP295, JP296, JP297, JP298, JP299, JP300: SEWTAP6, LilyPad-Wearables:PETAL-SMALL-2SIDE
- added LOGO100, LOGO52, LOGO54, LOGO56, LOGO58, LOGO60, LOGO62, LOGO64, LOGO66, LOGO68, LOGO70, LOGO72, LOGO74, LOGO76, LOGO78, LOGO80, LOGO82, LOGO84, LOGO86, LOGO88, LOGO90, LOGO92, LOGO94, LOGO96, LOGO98: SFE_LOGO_FLAME.1_INCH, SparkFun-Aesthetics:SFE_LOGO_FLAME_.1
- added LOGO51, LOGO53, LOGO55, LOGO57, LOGO59, LOGO61, LOGO63, LOGO65, LOGO67, LOGO69, LOGO71, LOGO73, LOGO75, LOGO77, LOGO79, LOGO81, LOGO83, LOGO85, LOGO87, LOGO89, LOGO91, LOGO93, LOGO95, LOGO97, LOGO99: OSHW-LOGOS, SparkFun-Aesthetics:OSHW-LOGO-S
- added U$100, U$52, U$54, U$56, U$58, U$60, U$62, U$64, U$66, U$68, U$70, U$72, U$74, U$76, U$78, U$80, U$82, U$84, U$86, U$88, U$90, U$92, U$94, U$96, U$98: LOGO-LPLP, LilyPad-Wearables:LOGO-LILYPAD
- added U$51, U$53, U$55, U$57, U$59, U$61, U$63, U$65, U$67, U$69, U$71, U$73, U$75, U$77, U$79, U$81, U$83, U$85, U$87, U$89, U$91, U$93, U$95, U$97, U$99: LOGO-LPL, LilyPad-Wearables:LOGO-L
Connections:
- new net DI26: D26.4, JP152.1, JP156.1
- new net DI27: D27.4, JP158.1, JP162.1
- new net DI28: D28.4, JP164.1, JP168.1
- new net DI29: D29.4, JP170.1, JP174.1
- new net DI30: D30.4, JP176.1, JP180.1
- new net DI31: D31.4, JP182.1, JP186.1
- new net DI32: D32.4, JP188.1, JP192.1
- new net DI33: D33.4, JP194.1, JP198.1
- new net DI34: D34.4, JP200.1, JP204.1
- new net DI35: D35.4, JP206.1, JP210.1
- new net DI36: D36.4, JP212.1, JP216.1
- new net DI37: D37.4, JP218.1, JP222.1
- new net DI38: D38.4, JP224.1, JP228.1
- new net DI39: D39.4, JP230.1, JP234.1
- new net DI40: D40.4, JP236.1, JP240.1
- new net DI41: D41.4, JP242.1, JP246.1
- new net DI42: D42.4, JP248.1, JP252.1
- new net DI43: D43.4, JP254.1, JP258.1
- new net DI44: D44.4, JP260.1, JP264.1
- new net DI45: D45.4, JP266.1, JP270.1
- new net DI46: D46.4, JP272.1, JP276.1
- new net DI47: D47.4, JP278.1, JP282.1
- new net DI48: D48.4, JP284.1, JP288.1
- new net DI49: D49.4, JP290.1, JP294.1
- new net DI50: D50.4, JP296.1, JP300.1
- new net DO26: D26.2, JP154.1, JP155.1
- new net DO27: D27.2, JP160.1, JP161.1
- new net DO28: D28.2, JP166.1, JP167.1
- new net DO29: D29.2, JP172.1, JP173.1
- new net DO30: D30.2, JP178.1, JP179.1
- new net DO31: D31.2, JP184.1, JP185.1
- new net DO32: D32.2, JP190.1, JP191.1
- new net DO33: D33.2, JP196.1, JP197.1
- new net DO34: D34.2, JP202.1, JP203.1
- new net DO35: D35.2, JP208.1, JP209.1
- new net DO36: D36.2, JP214.1, JP215.1
- new net DO37: D37.2, JP220.1, JP221.1
- new net DO38: D38.2, JP226.1, JP227.1
- new net DO39: D39.2, JP232.1, JP233.1
- new net DO40: D40.2, JP238.1, JP239.1
- new net DO41: D41.2, JP244.1, JP245.1
- new net DO42: D42.2, JP250.1, JP251.1
- new net DO43: D43.2, JP256.1, JP257.1
- new net DO44: D44.2, JP262.1, JP263.1
- new net DO45: D45.2, JP268.1, JP269.1
- new net DO46: D46.2, JP274.1, JP275.1
- new net DO47: D47.2, JP280.1, JP281.1
- new net DO48: D48.2, JP286.1, JP287.1
- new net DO49: D49.2, JP292.1, JP293.1
- new net DO50: D50.2, JP298.1, JP299.1
- new net GND25: C26.2, D26.3, JP153.1
- new net GND26: C27.2, D27.3, JP159.1
- new net GND27: C28.2, D28.3, JP165.1
- new net GND28: C29.2, D29.3, JP171.1
- new net GND29: C30.2, D30.3, JP177.1
- new net GND30: C31.2, D31.3, JP183.1
- new net GND31: C32.2, D32.3, JP189.1
- new net GND32: C33.2, D33.3, JP195.1
- new net GND33: C34.2, D34.3, JP201.1
- new net GND34: C35.2, D35.3, JP207.1
- new net GND35: C36.2, D36.3, JP213.1
- new net GND36: C37.2, D37.3, JP219.1
- new net GND37: C38.2, D38.3, JP225.1
- new net GND38: C39.2, D39.3, JP231.1
- new net GND39: C40.2, D40.3, JP237.1
- new net GND40: C41.2, D41.3, JP243.1
- new net GND41: C42.2, D42.3, JP249.1
- new net GND42: C43.2, D43.3, JP255.1
- new net GND43: C44.2, D44.3, JP261.1
- new net GND44: C45.2, D45.3, JP267.1
- new net GND45: C46.2, D46.3, JP273.1
- new net GND46: C47.2, D47.3, JP279.1
- new net GND47: C48.2, D48.3, JP285.1
- new net GND48: C49.2, D49.3, JP291.1
- new net GND49: C50.2, D50.3, JP297.1
- new net VCC25: C26.1, D26.1, JP151.1
- new net VCC26: C27.1, D27.1, JP157.1
- new net VCC27: C28.1, D28.1, JP163.1
- new net VCC28: C29.1, D29.1, JP169.1
- new net VCC29: C30.1, D30.1, JP175.1
- new net VCC30: C31.1, D31.1, JP181.1
- new net VCC31: C32.1, D32.1, JP187.1
- new net VCC32: C33.1, D33.1, JP193.1
- new net VCC33: C34.1, D34.1, JP199.1
- new net VCC34: C35.1, D35.1, JP205.1
- new net VCC35: C36.1, D36.1, JP211.1
- new net VCC36: C37.1, D37.1, JP217.1
- new net VCC37: C38.1, D38.1, JP223.1
- new net VCC38: C39.1, D39.1, JP229.1
- new net VCC39: C40.1, D40.1, JP235.1
- new net VCC40: C41.1, D41.1, JP241.1
- new net VCC41: C42.1, D42.1, JP247.1
- new net VCC42: C43.1, D43.1, JP253.1
- new net VCC43: C44.1, D44.1, JP259.1
- new net VCC44: C45.1, D45.1, JP265.1
- new net VCC45: C46.1, D46.1, JP271.1
- new net VCC46: C47.1, D47.1, JP277.1
- new net VCC47: C48.1, D48.1, JP283.1
- new net VCC48: C49.1, D49.1, JP289.1
- new net VCC49: C50.1, D50.1, JP295.1
Routing:
- net DO41: track 0.00 -> 17.7 mm
- net DO26: track 0.00 -> 17.7 mm
- net DO36: track 0.00 -> 17.7 mm
- net DO31: track 0.00 -> 17.7 mm
- net DO46: track 0.00 -> 17.7 mm
- net DO45: track 0.00 -> 17.7 mm
- net DO40: track 0.00 -> 17.7 mm
- net DO30: track 0.00 -> 17.7 mm
- net DO43: track 0.00 -> 17.7 mm
- net DO35: track 0.00 -> 17.7 mm
- net DO50: track 0.00 -> 17.7 mm
- net DO28: track 0.00 -> 17.7 mm
- net DO38: track 0.00 -> 17.7 mm
- net DO33: track 0.00 -> 17.7 mm
- net DO48: track 0.00 -> 17.7 mm
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- added copper zone on layer 1, net GND25
- added copper zone on layer 16, net GND25
- added copper zone on layer 1, net GND26
- added copper zone on layer 16, net GND26
- added copper zone on layer 1, net GND27
- added copper zone on layer 16, net GND27
- added copper zone on layer 1, net GND28
- added copper zone on layer 16, net GND28
- added copper zone on layer 1, net GND29
- added copper zone on layer 16, net GND29
- added copper zone on layer 1, net GND30
- added copper zone on layer 16, net GND30
- added copper zone on layer 1, net GND31
- added copper zone on layer 16, net GND31
- added copper zone on layer 1, net GND32
- added copper zone on layer 16, net GND32
- added copper zone on layer 1, net GND33
- added copper zone on layer 16, net GND33
- added copper zone on layer 1, net GND34
- added copper zone on layer 16, net GND34
- added copper zone on layer 1, net GND35
- added copper zone on layer 16, net GND35
- added copper zone on layer 1, net GND36
- added copper zone on layer 16, net GND36
- added copper zone on layer 1, net GND37
- added copper zone on layer 16, net GND37
- added copper zone on layer 1, net GND38
- added copper zone on layer 16, net GND38
- added copper zone on layer 1, net GND39
- added copper zone on layer 16, net GND39
- added copper zone on layer 1, net GND40
- added copper zone on layer 16, net GND40
- added copper zone on layer 1, net GND41
- added copper zone on layer 16, net GND41
- added copper zone on layer 1, net GND42
- added copper zone on layer 16, net GND42
- added copper zone on layer 1, net GND43
- added copper zone on layer 16, net GND43
- added copper zone on layer 1, net GND44
- added copper zone on layer 16, net GND44
- added copper zone on layer 1, net GND45
- added copper zone on layer 16, net GND45
- added copper zone on layer 1, net GND46
- added copper zone on layer 16, net GND46
- added copper zone on layer 1, net GND47
- added copper zone on layer 16, net GND47
- added copper zone on layer 1, net GND48
- added copper zone on layer 16, net GND48
- added copper zone on layer 1, net GND49
- added copper zone on layer 16, net GND49
Other:
- board size 129.5 x 129.5 mm -> 259.6 x 129.5 mm
